File: tria_hardware/TRIA_CentralControlBoard/can.kicad_sch (KiCad schematic)
At the start: 5 parts, among them J5 resistor_enable, U9 MCP2562-E-P

Commit message: [update] 基板データのアップデート
Other:
- moved on the sheet: C14, C15, J5, R17, U9
