File: tria_hardware/TRIA_ControlPowerBoard/TRIA_ControlPowerBoard.kicad_pcb (KiCad board)
At the start: 2 copper layers, 90 x 70 mm, 29 parts, among them J1 Batt, J10 out5V, J11 SW_LED, J2 out5V, J4 out5V, J6 power_swtich, J7 voltage_meter, J8 out5V, J9 out5V, Q1 MTP4835I3

Commit message: [update] 基板データのアップデート
Parts:
- renumbered J11 to LED, J6 to Main, J7 to Meter
Routing:
- net thermal: vias 8 -> 0
Changed lines of the file:
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@@
 			(outputformat 1)
 			(mirror no)
-			(drillshape 1)
+			(drillshape 0)
 			(scaleselection 1)
-			(outputdirectory "")
+			(outputdirectory "gerber/")
 		)
 	)
@@
 		(descr "JST XH series connector, B2B-XH-A (http://www.jst-mfg.com/product/pdf/eng/eXH.pdf), generated with kicad-footprint-generator")
 		(tags "connector JST XH vertical")
-		(property "Reference" "J11"
+		(property "Reference" "LED"
 			(at 1.25 -3.55 90)
 			(layer "F.SilkS")
@@
 		(descr "JST XH series connector, B2B-XH-A (http://www.jst-mfg.com/product/pdf/eng/eXH.pdf), generated with kicad-footprint-generator")
 		(tags "connector JST XH vertical")
-		(property "Reference" "J7"
+		(property "Reference" "Meter"
 			(at 1.25 -3.55 90)
 			(layer "F.SilkS")
@@
 		(descr "JST XH series connector, B2B-XH-A (http://www.jst-mfg.com/product/pdf/eng/eXH.pdf), generated with kicad-footprint-generator")
 		(tags "connector JST XH vertical")
-		(property "Reference" "J6"
+		(property "Reference" "Main"
 			(at 1.25 -3.55 90)
 			(layer "F.SilkS")
@@
 		(net 10)
 	)
-	(via
-		(at 72 77)
-		(size 0.6)
-		(drill 0.3)
-		(layers "F.Cu" "B.Cu")
-		(net 12)
-	)
-	(via
-		(at 73.5 78.5)
-		(size 0.6)
-		(drill 0.3)
-		(layers "F.Cu" "B.Cu")
-		(net 12)
-	)
-	(via
-		(at 72 75.5)
-		(size 0.6)
-		(drill 0.3)
-		(layers "F.Cu" "B.Cu")
-		(net 12)
-	)
-	(via
-		(at 79.5 78.5)
-		(size 0.6)
-		(drill 0.3)
-		(layers "F.Cu" "B.Cu")
-		(net 12)
-	)
-	(via
-		(at 78 78.5)
-		(size 0.6)
-		(drill 0.3)
-		(layers "F.Cu" "B.Cu")
-		(net 12)
-	)
-	(via
-		(at 72 78.5)
-		(size 0.6)
-		(drill 0.3)
-		(layers "F.Cu" "B.Cu")
-		(net 12)
-	)
-	(via
-		(at 76.5 78.5)
-		(size 0.6)
-		(drill 0.3)
-		(layers "F.Cu" "B.Cu")
-		(net 12)
-	)
-	(via
-		(at 75 78.5)
-		(size 0.6)
-		(drill 0.3)
-		(layers "F.Cu" "B.Cu")
-		(net 12)
-	)
 	(zone
