File: tria_hardware/TRIA_DrivePowerBoard/TRIA_DrivePowerBoard.kicad_pcb (KiCad board)
At the start: 2 copper layers, 90 x 70 mm, 23 parts, among them J10 out, J11 out, J12 out, J3 out, J4 out, J5 out, J8 out, J9 out, Q1 MTP4835I3, Q2 MTP4835I3

Commit message: [update] 基板データのアップデート
Routing:
- net (no net): vias 12 -> 0
Changed lines of the file:
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@@
 			(outputformat 1)
 			(mirror no)
-			(drillshape 1)
+			(drillshape 0)
 			(scaleselection 1)
-			(outputdirectory "")
+			(outputdirectory "gerber/")
 		)
 	)
@@
 		)
 	)
-	(via
-		(at 88.5 71.5)
-		(size 0.6)
-		(drill 0.3)
-		(layers "F.Cu" "B.Cu")
-		(free yes)
-		(net 0)
-	)
-	(via
-		(at 110 71.5)
-		(size 0.6)
-		(drill 0.3)
-		(layers "F.Cu" "B.Cu")
-		(free yes)
-		(net 0)
-	)
-	(via
-		(at 108.5 71.5)
-		(size 0.6)
-		(drill 0.3)
-		(layers "F.Cu" "B.Cu")
-		(free yes)
-		(net 0)
-	)
-	(via
-		(at 105.5 71.5)
-		(size 0.6)
-		(drill 0.3)
-		(layers "F.Cu" "B.Cu")
-		(free yes)
-		(net 0)
-	)
-	(via
-		(at 107 71.5)
-		(size 0.6)
-		(drill 0.3)
-		(layers "F.Cu" "B.Cu")
-		(free yes)
-		(net 0)
-	)
-	(via
-		(at 84 71.5)
-		(size 0.6)
-		(drill 0.3)
-		(layers "F.Cu" "B.Cu")
-		(free yes)
-		(net 0)
-	)
-	(via
-		(at 91.5 71.5)
-		(size 0.6)
-		(drill 0.3)
-		(layers "F.Cu" "B.Cu")
-		(free yes)
-		(net 0)
-	)
-	(via
-		(at 85.5 71.5)
-		(size 0.6)
-		(drill 0.3)
-		(layers "F.Cu" "B.Cu")
-		(free yes)
-		(net 0)
-	)
-	(via
-		(at 90 71.5)
-		(size 0.6)
-		(drill 0.3)
-		(layers "F.Cu" "B.Cu")
-		(free yes)
-		(net 0)
-	)
-	(via
-		(at 111.5 71.5)
-		(size 0.6)
-		(drill 0.3)
-		(layers "F.Cu" "B.Cu")
-		(free yes)
-		(net 0)
-	)
-	(via
-		(at 87 71.5)
-		(size 0.6)
-		(drill 0.3)
-		(layers "F.Cu" "B.Cu")
-		(free yes)
-		(net 0)
-	)
-	(via
-		(at 104 71.5)
-		(size 0.6)
-		(drill 0.3)
-		(layers "F.Cu" "B.Cu")
-		(free yes)
-		(net 0)
-	)
 	(segment
