File: tria_hardware/TRIA_MotorDrive/TRIA_MotorDrive.kicad_pcb (KiCad board)
At the start: 2 copper layers, 90 x 70 mm, 62 parts, among them J1 PowerBatt, J2 LogicBatt, J3 encoder, J4 CAN, J5 resistor_enable, M1 Motor_DC, Q1 MTB7D0N06RJ3, Q2 LOW1, Q3 HIGH2, Q4 LOW2, SW1 SW_Push, SW2 SW_Push, U1 IR2302, U2 IR2302, U3 ACS711xLCTR-12AB, U4 M78AR12-0.5, U5 SeeeduinoXIAO, U6 PC817, U7 TA78L05S, U8 PC817, U9 MCP2562-E-P

Commit message: [update] 基板データのアップデート
Parts:
- removed C12, C13, C17: 0.1u, Capacitor_THT:C_Disc_D3.0mm_W1.6mm_P2.50mm
- removed C2: 1u, Capacitor_THT:C_Disc_D3.0mm_W1.6mm_P2.50mm
- removed D1, D2: 1N5819, Diode_THT:D_DO-41_SOD81_P7.62mm_Horizontal
- removed D3, D4: LED, LED_THT:LED_D3.0mm
- removed M1: Motor_DC, Connector_AMASS:AMASS_XT60-F_1x02_P7.20mm_Vertical
- removed Q1: MTB7D0N06RJ3, Package_TO_SOT_SMD:TO-252-2
- removed Q2: LOW1, Package_TO_SOT_SMD:TO-252-2
- removed Q3: HIGH2, Package_TO_SOT_SMD:TO-252-2
- removed Q4: LOW2, Package_TO_SOT_SMD:TO-252-2
- removed R10, R9: 10k, Resistor_THT:R_Axial_DIN0207_L6.3mm_D2.5mm_P10.16mm_Horizontal
- removed R3, R4, R7, R8: 10k, Resistor_SMD:R_1206_3216Metric_Pad1.30x1.75mm_HandSolder
- removed R5, R6: 10, Resistor_SMD:R_1206_3216Metric_Pad1.30x1.75mm_HandSolder
- removed U1, U2: IR2302, Package_SO:SOIC-8_3.9x4.9mm_P1.27mm
- removed U3: ACS711xLCTR-12AB, Package_SO:SOIC-8_3.9x4.9mm_P1.27mm
- added C5: 0.1u, Capacitor_THT:C_Disc_D3.0mm_W1.6mm_P2.50mm, F.Cu at (92.7, 61.2)
- added M2: Motor_DC, Connector_AMASS:AMASS_XT60-F_1x02_P7.20mm_Vertical, F.Cu at (110.0, 100.0)
- added PWM1: LED, LED_THT:LED_D3.0mm, F.Cu at (144.0, 94.0)
- added PWM2: LED, LED_THT:LED_D3.0mm, F.Cu at (150.0, 94.0)
- added U10: TB67H450FNG_EL, footprints:P-HSOP8-0405-1p27-002_TOS, F.Cu at (90.0, 65.0)
- C1: value 1u -> 10uF16V; footprint Capacitor_THT:C_Disc_D3.0mm_W1.6mm_P2.50mm -> Capacitor_THT:CP_Radial_D4.0mm_P1.50mm
- C3: value 0.1u -> 100uF50V; footprint Capacitor_THT:C_Disc_D3.0mm_W1.6mm_P2.50mm -> Capacitor_THT:CP_Radial_D8.0mm_P3.50mm
- R1, R2: value 10 -> 10k; footprint Resistor_SMD:R_1206_3216Metric_Pad1.30x1.75mm_HandSolder -> Resistor_THT:R_Axial_DIN0207_L6.3mm_D2.5mm_P10.16mm_Horizontal
- R11: value PullUp -> 10k
- R12: value 1k -> 10k
- U7: value TA78L05S -> LP2950L-33-T92
- moved R2 61.6 mm to (139.0, 63.0)
- moved C3 59.7 mm to (87.3, 55.2), turned to 0 degrees
- moved R21 58.0 mm to (139.0, 106.5), turned to 90 degrees
- moved R1 56.4 mm to (139.0, 66.1)
- moved R20 53.4 mm to (139.0, 100.5), turned to 90 degrees
- moved C4 50.3 mm to (87.3, 61.1), turned to 0 degrees
- moved C9 40.0 mm to (112.5, 72.2), turned to 180 degrees
- moved R12 36.2 mm to (99.3, 75.8), turned to 90 degrees
- moved D5 35.9 mm to (117.6, 58.4), turned to -90 degrees
- moved C8 35.7 mm to (112.5, 68.2), turned to 180 degrees
- moved R11 33.3 mm to (95.3, 75.8), turned to 90 degrees
- moved U4 32.6 mm to (110.0, 65.0), turned to 0 degrees
- moved C16 32.4 mm to (113.0, 77.0), turned to 180 degrees
- moved U7 32.0 mm to (113.0, 80.0), turned to 180 degrees
- moved J3 28.0 mm to (121.0, 80.0)
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Connections:
- C1 pad 1: Net-(D1-K) -> +3.3V
- C1 pad 2: /MotorDrive/CurrentSensor/IP+ -> GND
- C14 pad 1: +3.3V -> +3.3VD
- C3 pad 1: /MPU/CurrentSensor -> +BATT
- C3 pad 2: GNDD -> GND
- C4 pad 1: VDD -> +BATT
- C4 pad 2: GNDD -> GND
- J4 pad 1: /CAN/CAN_H -> /CAN/CAN_L
- J4 pad 2: /CAN/CAN_L -> /CAN/CAN_H
- R1 pad 1: Net-(U1-HO) -> GNDD
- R1 pad 2: Net-(Q1-G) -> Net-(U5-PA4_A1_D1)
- R11 pad 1: Net-(U3-~{FAULT}) -> GND
- R11 pad 2: VDD -> /MotorDrive/PWM2
- R12 pad 1: /MPU/CurrentSensor -> GND
- R12 pad 2: Net-(U3-VIOUT) -> /MotorDrive/PWM1
- R14 pad 1: +5V -> +3.3V
- R16 pad 1: +5V -> +3.3V
- R2 pad 1: Net-(U1-LO) -> GNDD
- R2 pad 2: Net-(Q2-G) -> Net-(U5-PA02_A0_D0)
- R20 pad 2: /MotorDrive/PWM1 -> /MPU/pwm1
- R21 pad 2: /MotorDrive/PWM2 -> /MPU/pwm2
- SW1 pad 1: unconnected-(SW1-Pad1) -> +3.3VD
- SW1 pad 2: unconnected-(SW1-Pad2) -> Net-(U5-PA02_A0_D0)
- SW2 pad 1: unconnected-(SW2-Pad1) -> +3.3VD
- SW2 pad 2: unconnected-(SW2-Pad2) -> Net-(U5-PA4_A1_D1)
- U5 pad 1: unconnected-(U5-PA02_A0_D0-Pad1) -> Net-(U5-PA02_A0_D0)
- U5 pad 10: unconnected-(U5-PA5_A9_D9_MISO-Pad10) -> /MPU/pwm1
- U5 pad 11: unconnected-(U5-PA6_A10_D10_MOSI-Pad11) -> /MPU/pwm2
- U5 pad 12: +3.3V -> +3.3VD
- U5 pad 2: unconnected-(U5-PA4_A1_D1-Pad2) -> Net-(U5-PA4_A1_D1)
- U5 pad 3: unconnected-(U5-PA10_A2_D2-Pad3) -> /MPU/ENCODER_B
- U5 pad 4: unconnected-(U5-PA11_A3_D3-Pad4) -> /MPU/ENCODER_A
- U5 pad 5: unconnected-(U5-PA8_A4_D4_SDA-Pad5) -> /CAN/CAN_RX
- U5 pad 6: unconnected-(U5-PA9_A5_D5_SCL-Pad6) -> /CAN/CAN_TX
- U7 pad 3: +5V -> +3.3V
- U9 pad 5: +3.3V -> +3.3VD
Routing:
- net +5V: track 84.4 -> 0.00 mm
- net +3.3VD: track 0.00 -> 56.3 mm
- net +12V: track 74.5 -> 20.7 mm
- net +BATT: track 22.1 -> 71.4 mm
- net /MotorDrive/CurrentSensor/IP+: track 48.5 -> 0.00 mm
- net /MotorDrive/PWM2: track 105.6 -> 59.5 mm
- net Net-(Q1-G): track 45.7 -> 0.00 mm, vias 2 -> 0
- net GNDD: track 45.1 -> 2.94 mm
- net /MotorDrive/PWM1: track 97.6 -> 64.5 mm
- net Net-(Q2-G): track 30.0 -> 0.00 mm, vias 2 -> 0
- net VDD: track 157.6 -> 130.3 mm
- net Net-(U3-VIOUT): track 22.4 -> 0.00 mm
- net Net-(U3-~{FAULT}): track 21.4 -> 0.00 mm
- net Net-(U2-VS): track 21.1 -> 0.00 mm
- net /MPU/ENCODER_B: track 9.04 -> 30.2 mm
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- added copper zone on F.Cu, net GND
- added copper zone on F.Cu, net Net-(M2-+)
- added copper zone on F.Cu, net Net-(M2--)
- removed copper zone on F.Cu, net +BATT
- removed copper zone on F.Cu, net /MotorDrive/CurrentSensor/IP+
- removed copper zone on F.Cu, net /MotorDrive/CurrentSensor/IP-
- removed copper zone on B.Cu, net GND
- removed copper zone on F.Cu, net Net-(M1--)
Other:
- board text added: "Board Size 90 x 70 Distance Between holes 80 x 60"
- board text added: "Encoder PIN A B VDD GND"
- board text removed: "A"
- board text removed: "B"
- board text removed: "GND"
- board text removed: "VDD"
