File: tria_hardware/TRIA_MotorDrive/TRIA_MotorDrive.kicad_sch (KiCad schematic)
At the start: 15 parts, among them J1 PowerBatt, J2 LogicBatt, J3 encoder, J4 CAN, U4 M78AR12-0.5, U7 TA78L05S

Commit message: [update] 基板データのアップデート
Parts:
- removed C17: 0.1u, Capacitor_THT:C_Disc_D3.0mm_W1.6mm_P2.50mm, symbol Device:C
- added C1: 10uF16V, Capacitor_THT:CP_Radial_D4.0mm_P1.50mm, symbol Device:C_Polarized
- U7: value TA78L05S -> LP2950L-33-T92
Connections:
- net CAN/CAN_H: now also J4.2 (Pin_2); no longer J4.1 (Pin_1)
- net CAN/CAN_L: now also J4.1 (Pin_1); no longer J4.2 (Pin_2)
- net GND: now also C1.2
- net +5V renamed +3.3V
- net +3.3V: now also C1.1
Other:
- sheet MPU ports: added none; removed CurrentSensor
- sheet MotorDrive ports: added none; removed CurrentSensor
- moved on the sheet: J4
