File: tria_hardware/TRIA_MotorDrive/photo_coupler.kicad_sch (KiCad schematic)
At the start: 10 parts, among them U6 PC817, U8 PC817

Commit message: [update] 基板データのアップデート
Connections:
- net GND: no longer D3.1 (K), D4.1 (K)
- net GNDD: now also D3.1 (K), D4.1 (K)
- net pwm1_in: now also R20.2
- net pwm1_out: no longer R20.2
- net pwm2_in: now also R21.2
- net pwm2_out: no longer R21.2
- net +5V renamed +3.3V
Other:
- moved on the sheet: D3, D4, R20, R21
